Commit message: Added tables, adjusted panda_simulation launch file to spawn objects.

File: sdf/pudding_box/pudding_box.urdf (robot description, URDF)
Before this commit: robot Pudding Box, 2 links, 1 joints
Links:
- removed link world
- link pudding_box: geometry collision mesh filename=package://sdf/pudding_box/textured.dae scale=1 1 1; visual mesh filename=package://sdf/pudding_box/textured.dae scale=1 1 1
Joints:
- removed joint fixed
